File: circuit/elekey.brd (EAGLE design)
At the start: 52.1 x 29.2 mm, 22 parts, among them Q1 2N7000, Q2 2N7000, X1 PG203J

Commit message: コメントがおかしい
Parts:
- removed R1, R2: VARISTOR-2,5, varistor:R-5
- added D1, D2: 3.3V, diode:ZDIO-5
- IC1: value TINY2313-*P* -> ATTiny2313
- SG1: value EFBRD24C411 -> (none)
- X1: value PG203J -> (none)
- moved SG1 51.7 mm to (63.5, 36.8), turned to 180 degrees
- moved JP2 15.3 mm to (35.6, 26.7), turned to 90 degrees
- moved R3 12.7 mm to (30.5, 25.4)
- moved C2 12.7 mm to (33.0, 25.4)
- moved Q1 10.2 mm to (27.9, 25.4)
- renumbered U$1 to IC1
Connections:
- net GND: now also D1.A, D2.A; no longer R1.1, R2.1
- net N$1: now also D1.C; no longer R2.2
- net N$2: now also D2.C; no longer R1.2
Routing:
- net N$9: track 20.3 -> 7.62 mm
- net N$8: track 38.1 -> 35.6 mm
- net N$1: track 32.8 -> 30.6 mm
- net N$2: track 36.5 -> 35.7 mm
