File: circuit/elekey.sch (EAGLE design)
At the start: 22 parts, among them Q1 2N7000, Q2 2N7000, X1 PG203J

Commit message: コメントがおかしい
Parts:
- removed R1, R2: VARISTOR-2,5, varistor:VARISTOR-2,5
- added D1, D2: 3.3V, diode:ZENER-DIODEZD-5
- IC1: value TINY2313-*P* -> ATTiny2313
- renumbered U$1 to IC1
Connections:
- net GND: now also D1.A, D2.A; no longer R1.1, R2.1
- net N$1: now also D1.C; no longer R2.2
- net N$2: now also D2.C; no longer R1.2
Other:
- moved on the sheet: JP5
